File: rev2/Plates/hull/hull.kicad_pcb (KiCad board)
At the start: 2 copper layers, 251.2 x 76.2 mm, 44 parts

Commit message: Fix plate encoder cutouts
Other:
- outline, holes or cut-outs redrawn
Changed lines of the file:
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@@
     (visible_elements 7FFFEFFF)
     (pcbplotparams
-      (layerselection 0x010f0_ffffffff)
+      (layerselection 0x010c0_ffffffff)
       (usegerberextensions false)
       (usegerberattributes false)
@@
       (drillshape 0)
       (scaleselection 1)
-      (outputdirectory ""))
+      (outputdirectory "./"))
   )
   (net 0 "")
@@
     (fp_line (start -16.66875 9.525) (end -16.66875 -9.525) (layer Dwgs.User) (width 0.15))
     (fp_line (start -16.66875 -9.525) (end 16.66875 -9.525) (layer Dwgs.User) (width 0.15))
-    (fp_line (start 13.64375 -7) (end -13.64375 -7) (layer Edge.Cuts) (width 0.05))
+    (fp_line (start 15.33125 -7) (end -13.64375 -7) (layer Edge.Cuts) (width 0.05))
     (fp_line (start -14.14375 -6.5) (end -14.14375 6.5) (layer Edge.Cuts) (width 0.05))
-    (fp_line (start -13.64375 7) (end 13.64375 7) (layer Edge.Cuts) (width 0.05))
-    (fp_line (start 14.14375 6.5) (end 14.14375 -6.5) (layer Edge.Cuts) (width 0.05))
-    (fp_arc (start 13.64375 -6.5) (end 14.14375 -6.5) (angle -90) (layer Edge.Cuts) (width 0.05))
+    (fp_line (start -13.64375 7) (end 15.33125 7) (layer Edge.Cuts) (width 0.05))
+    (fp_line (start 15.83125 6.5) (end 15.83125 -6.5) (layer Edge.Cuts) (width 0.05))
+    (fp_arc (start 15.33125 -6.5) (end 15.83125 -6.5) (angle -90) (layer Edge.Cuts) (width 0.05))
     (fp_arc (start -13.64375 -6.5) (end -13.64375 -7) (angle -90) (layer Edge.Cuts) (width 0.05))
     (fp_arc (start -13.64375 6.5) (end -14.14375 6.5) (angle -90) (layer Edge.Cuts) (width 0.05))
-    (fp_arc (start 13.64375 6.5) (end 13.64375 7) (angle -90) (layer Edge.Cuts) (width 0.05))
-    (pad 1 smd roundrect (at 0 0 180) (size 30.2875 16) (layers F.Cu F.Mask) (roundrect_rratio 0.063))
-    (pad 1 smd roundrect (at 0 0 180) (size 30.2875 16) (layers B.Cu B.Mask) (roundrect_rratio 0.063))
+    (fp_arc (start 15.33125 6.5) (end 15.33125 7) (angle -90) (layer Edge.Cuts) (width 0.05))
+    (pad 1 smd roundrect (at 0.84375 0 180) (size 31.975 16) (layers F.Cu F.Mask) (roundrect_rratio 0.063))
+    (pad 1 smd roundrect (at 0.84375 0 180) (size 31.975 16) (layers B.Cu B.Mask) (roundrect_rratio 0.063))
   )
   (module Keybage_MX_Cutout:MX_Cutout_3u (layer F.Cu)
@@
   (gr_arc (start 10.311779 88.793401) (end 10.31178 86.118401) (angle -37.87921967) (layer Edge.Cuts) (width 0.2))
   (gr_arc (start 8.63678 17.943401) (end 8.879317 19.169645) (angle -157.6238886) (layer Edge.Cuts) (width 0.2))
-  (gr_line (start 255.52428 84.618401) (end 255.52428 22.118401) (layer Edge.Cuts) (width 0.2))
+  (gr_line (start 255.52428 84.6184) (end 255.52428 22.118401) (layer Edge.Cuts) (width 0.2))
   (gr_arc (start 257.02428 84.6184) (end 255.52428 84.6184) (angle -90) (layer Edge.Cuts) (width 0.2))
   (gr_arc (start 259.184727 87.076658) (end 259.281742 87.567156) (angle -130.9327246) (layer Edge.Cuts) (width 0.2))
-  (gr_arc (start 257.84928 17.943401) (end 257.84928 20.618401) (angle -37.87921967) (layer Edge.Cuts) (width 0.2))
-  (gr_line (start 11.13678 86.118401) (end 10.311779 86.118401) (layer Edge.Cuts) (width 0.2))
+  (gr_arc (start 257.849283 17.9434) (end 257.849283 20.6184) (angle -37.87921967) (layer Edge.Cuts) (width 0.2))
+  (gr_line (start 11.13678 86.118401) (end 10.31178 86.118401) (layer Edge.Cuts) (width 0.2))
   (gr_arc (start 257.84928 88.793401) (end 257.84928 91.468401) (angle -37.87921967) (layer Edge.Cuts) (width 0.2))
-  (gr_line (start 257.02428 20.618401) (end 257.84928 20.618401) (layer Edge.Cuts) (width 0.2))
+  (gr_line (start 257.02428 20.618401) (end 257.849283 20.6184) (layer Edge.Cuts) (width 0.2))
   (gr_arc (start 257.02428 22.118401) (end 257.02428 20.618401) (angle -90) (layer Edge.Cuts) (width 0.2))
   (gr_arc (start 8.976332 87.076658) (end 8.669332 86.682005) (angle -130.9327246) (layer Edge.Cuts) (width 0.2))
   (gr_arc (start 10.311779 88.793401) (end 8.669332 90.904796) (angle -37.87921967) (layer Edge.Cuts) (width 0.2))
-  (gr_arc (start 259.52428 17.9434) (end 259.281742 16.717156) (angle -157.6238885) (layer Edge.Cuts) (width 0.2))
-  (gr_arc (start 259.184727 19.660143) (end 259.491727 20.054796) (angle -130.9327246) (layer Edge.Cuts) (width 0.2))
-  (gr_line (start 257.84928 86.118401) (end 257.02428 86.118401) (layer Edge.Cuts) (width 0.2))
+  (gr_arc (start 259.52428 17.943401) (end 259.281742 16.717157) (angle -157.6238885) (layer Edge.Cuts) (width 0.2))
+  (gr_arc (start 259.18473 19.660143) (end 259.49173 20.054796) (angle -130.9327246) (layer Edge.Cuts) (width 0.2))
+  (gr_line (start 257.84928 86.118401) (end 257.02428 86.1184) (layer Edge.Cuts) (width 0.2))
   (gr_arc (start 10.31178 17.9434) (end 8.669332 20.054796) (angle -37.87921966) (layer Edge.Cuts) (width 0.2))
   (gr_arc (start 8.976332 19.660143) (end 8.879317 19.169645) (angle -130.9327246) (layer Edge.Cuts) (width 0.2))
   (gr_arc (start 8.976332 16.226658) (end 8.669332 15.832005) (angle -130.9327246) (layer Edge.Cuts) (width 0.2))
-  (gr_line (start 10.311779 91.468401) (end 257.84928 91.468401) (layer Edge.Cuts) (width 0.2))
+  (gr_line (start 10.311779 91.4684) (end 257.84928 91.468401) (layer Edge.Cuts) (width 0.2))
   (gr_line (start 10.31178 20.618401) (end 11.13678 20.618401) (layer Edge.Cuts) (width 0.2))
-  (gr_line (start 12.63678 22.118401) (end 12.636779 84.618401) (layer Edge.Cuts) (width 0.2))
+  (gr_line (start 12.63678 22.118401) (end 12.63678 84.618401) (layer Edge.Cuts) (width 0.2))
   (gr_arc (start 11.13678 22.118401) (end 12.63678 22.118401) (angle -90) (layer Edge.Cuts) (width 0.2))
   (gr_arc (start 10.31178 17.9434) (end 10.311779 15.268401) (angle -37.87921973) (layer Edge.Cuts) (width 0.2))
@@
   (gr_line (start 257.84928 15.268401) (end 10.311779 15.268401) (layer Edge.Cuts) (width 0.2))
   (gr_arc (start 257.84928 17.943401) (end 259.491727 15.832005) (angle -37.87921967) (layer Edge.Cuts) (width 0.2))
-  (gr_arc (start 259.184727 16.226658) (end 259.281742 16.717156) (angle -130.9327246) (layer Edge.Cuts) (width 0.2))
+  (gr_arc (start 259.184727 16.226659) (end 259.281742 16.717157) (angle -130.9327246) (layer Edge.Cuts) (width 0.2))
 )
