File: rev2/Plates/minivan/minivan.kicad_pcb (KiCad board)
At the start: 2 copper layers, 243.4 x 76.2 mm, 50 parts

Commit message: Fix plate encoder cutouts
Changed lines of the file:
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@@
     (visible_elements 7FFFEFFF)
     (pcbplotparams
-      (layerselection 0x010f0_ffffffff)
+      (layerselection 0x010c0_ffffffff)
       (usegerberextensions false)
       (usegerberattributes false)
@@
       (drillshape 0)
       (scaleselection 1)
-      (outputdirectory ""))
+      (outputdirectory "./"))
   )
   (net 0 "")
@@
     (uvia_dia 0.3)
     (uvia_drill 0.1)
+  )
+  (module Keybage_MX_Cutout:MX_Cutout_1.75u_enc (layer F.Cu)
+    (at 238.9037 24.6047)
+    (fp_text reference REF** (at 0.25 10.05) (layer Eco2.User) hide
+      (effects (font (size 1 1) (thickness 0.15)))
+    )
+    (fp_text value MX_Cutout_1.75u_enc (at 0 -15.24) (layer F.Fab) hide
+      (effects (font (size 1 1) (thickness 0.15)))
+    )
+    (fp_line (start 16.66875 -9.525) (end 16.66875 9.525) (layer Dwgs.User) (width 0.15))
+    (fp_line (start 16.66875 9.525) (end -16.66875 9.525) (layer Dwgs.User) (width 0.15))
+    (fp_line (start -16.66875 9.525) (end -16.66875 -9.525) (layer Dwgs.User) (width 0.15))
+    (fp_line (start -16.66875 -9.525) (end 16.66875 -9.525) (layer Dwgs.User) (width 0.15))
+    (fp_line (start 15.33125 -7) (end -13.64375 -7) (layer Edge.Cuts) (width 0.05))
+    (fp_line (start -14.14375 -6.5) (end -14.14375 6.5) (layer Edge.Cuts) (width 0.05))
+    (fp_line (start -13.64375 7) (end 15.33125 7) (layer Edge.Cuts) (width 0.05))
+    (fp_line (start 15.83125 6.5) (end 15.83125 -6.5) (layer Edge.Cuts) (width 0.05))
+    (fp_arc (start 15.33125 -6.5) (end 15.83125 -6.5) (angle -90) (layer Edge.Cuts) (width 0.05))
+    (fp_arc (start -13.64375 -6.5) (end -13.64375 -7) (angle -90) (layer Edge.Cuts) (width 0.05))
+    (fp_arc (start -13.64375 6.5) (end -14.14375 6.5) (angle -90) (layer Edge.Cuts) (width 0.05))
+    (fp_arc (start 15.33125 6.5) (end 15.33125 7) (angle -90) (layer Edge.Cuts) (width 0.05))
+    (pad 1 smd roundrect (at 0.84375 0 180) (size 31.975 16) (layers F.Cu F.Mask) (roundrect_rratio 0.063))
+    (pad 1 smd roundrect (at 0.84375 0 180) (size 31.975 16) (layers B.Cu B.Mask) (roundrect_rratio 0.063))
   )
   (module Project-Parts:platehole (layer F.Cu)
@@
     (pad "" np_thru_hole circle (at 0 0) (size 6 6) (drill 5.1) (layers *.Cu *.Mask))
   )
-  (module Keybage_MX_Cutout:MX_Cutout_1.75u_enc (layer F.Cu)
-    (at 238.9037 24.6047)
-    (fp_text reference REF** (at 0.25 10.05) (layer Eco2.User) hide
-      (effects (font (size 1 1) (thickness 0.15)))
-    )
-    (fp_text value MX_Cutout_1.75u_enc (at 0 -15.24) (layer F.Fab) hide
-      (effects (font (size 1 1) (thickness 0.15)))
-    )
-    (fp_line (start 16.66875 -9.525) (end 16.66875 9.525) (layer Dwgs.User) (width 0.15))
-    (fp_line (start 16.66875 9.525) (end -16.66875 9.525) (layer Dwgs.User) (width 0.15))
-    (fp_line (start -16.66875 9.525) (end -16.66875 -9.525) (layer Dwgs.User) (width 0.15))
-    (fp_line (start -16.66875 -9.525) (end 16.66875 -9.525) (layer Dwgs.User) (width 0.15))
-    (fp_line (start 13.64375 -7) (end -13.64375 -7) (layer Edge.Cuts) (width 0.05))
-    (fp_line (start -14.14375 -6.5) (end -14.14375 6.5) (layer Edge.Cuts) (width 0.05))
-    (fp_line (start -13.64375 7) (end 13.64375 7) (layer Edge.Cuts) (width 0.05))
-    (fp_line (start 14.14375 6.5) (end 14.14375 -6.5) (layer Edge.Cuts) (width 0.05))
-    (fp_arc (start 13.64375 -6.5) (end 14.14375 -6.5) (angle -90) (layer Edge.Cuts) (width 0.05))
-    (fp_arc (start -13.64375 -6.5) (end -13.64375 -7) (angle -90) (layer Edge.Cuts) (width 0.05))
-    (fp_arc (start -13.64375 6.5) (end -14.14375 6.5) (angle -90) (layer Edge.Cuts) (width 0.05))
-    (fp_arc (start 13.64375 6.5) (end 13.64375 7) (angle -90) (layer Edge.Cuts) (width 0.05))
-    (pad 1 smd roundrect (at 0 0 180) (size 30.2875 16) (layers F.Cu F.Mask) (roundrect_rratio 0.063))
-    (pad 1 smd roundrect (at 0 0 180) (size 30.2875 16) (layers B.Cu B.Mask) (roundrect_rratio 0.063))
-  )
   (module Keybage_MX_Cutout:MX_Cutout_3u (layer F.Cu)
