File: rev2/Plates/p3d-topmount/p3d-topmount.kicad_pcb (KiCad board)
At the start: 2 copper layers, 257.1 x 90.4 mm, 44 parts

Commit message: Fix plate encoder cutouts
Other:
- outline, holes or cut-outs redrawn
Changed lines of the file:
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@@
     (visible_elements 7FFFEFFF)
     (pcbplotparams
-      (layerselection 0x010f0_ffffffff)
+      (layerselection 0x010c0_ffffffff)
       (usegerberextensions false)
       (usegerberattributes false)
@@
     (fp_line (start -16.66875 9.525) (end -16.66875 -9.525) (layer Dwgs.User) (width 0.15))
     (fp_line (start -16.66875 -9.525) (end 16.66875 -9.525) (layer Dwgs.User) (width 0.15))
-    (fp_line (start 13.64375 -7) (end -13.64375 -7) (layer Edge.Cuts) (width 0.05))
+    (fp_line (start 15.33125 -7) (end -13.64375 -7) (layer Edge.Cuts) (width 0.05))
     (fp_line (start -14.14375 -6.5) (end -14.14375 6.5) (layer Edge.Cuts) (width 0.05))
-    (fp_line (start -13.64375 7) (end 13.64375 7) (layer Edge.Cuts) (width 0.05))
-    (fp_line (start 14.14375 6.5) (end 14.14375 -6.5) (layer Edge.Cuts) (width 0.05))
-    (fp_arc (start 13.64375 -6.5) (end 14.14375 -6.5) (angle -90) (layer Edge.Cuts) (width 0.05))
+    (fp_line (start -13.64375 7) (end 15.33125 7) (layer Edge.Cuts) (width 0.05))
+    (fp_line (start 15.83125 6.5) (end 15.83125 -6.5) (layer Edge.Cuts) (width 0.05))
+    (fp_arc (start 15.33125 -6.5) (end 15.83125 -6.5) (angle -90) (layer Edge.Cuts) (width 0.05))
     (fp_arc (start -13.64375 -6.5) (end -13.64375 -7) (angle -90) (layer Edge.Cuts) (width 0.05))
     (fp_arc (start -13.64375 6.5) (end -14.14375 6.5) (angle -90) (layer Edge.Cuts) (width 0.05))
-    (fp_arc (start 13.64375 6.5) (end 13.64375 7) (angle -90) (layer Edge.Cuts) (width 0.05))
-    (pad 1 smd roundrect (at 0 0 180) (size 30.2875 16) (layers F.Cu F.Mask) (roundrect_rratio 0.063))
-    (pad 1 smd roundrect (at 0 0 180) (size 30.2875 16) (layers B.Cu B.Mask) (roundrect_rratio 0.063))
+    (fp_arc (start 15.33125 6.5) (end 15.33125 7) (angle -90) (layer Edge.Cuts) (width 0.05))
+    (pad 1 smd roundrect (at 0.84375 0 180) (size 31.975 16) (layers F.Cu F.Mask) (roundrect_rratio 0.063))
+    (pad 1 smd roundrect (at 0.84375 0 180) (size 31.975 16) (layers B.Cu B.Mask) (roundrect_rratio 0.063))
   )
   (module Keybage_MX_Cutout:MX_Cutout_3u (layer F.Cu)
@@
   (gr_line (start 191.551119 9.901555) (end 191.055048 11.433691) (layer Edge.Cuts) (width 0.2))
   (gr_arc (start 8.39584 53.171654) (end 7.525644 50.484019) (angle -144.118436) (layer Edge.Cuts) (width 0.2))
-  (gr_circle (center 7.89584 53.171654) (end 8.82084 53.171654) (layer Edge.Cuts) (width 0.2))
-  (gr_circle (center 260.383754 53.171654) (end 261.308754 53.171654) (layer Edge.Cuts) (width 0.2))
-  (gr_circle (center 194.238754 10.271751) (end 195.163754 10.271751) (layer Edge.Cuts) (width 0.2))
-  (gr_circle (center 74.04084 10.271751) (end 74.96584 10.271751) (layer Edge.Cuts) (width 0.2))
-  (gr_circle (center 74.04084 96.071557) (end 74.96584 96.071557) (layer Edge.Cuts) (width 0.2))
-  (gr_circle (center 194.238754 96.071557) (end 195.163754 96.071557) (layer Edge.Cuts) (width 0.2))
+  (gr_circle (center 7.89584 53.171654) (end 8.89584 53.171654) (layer Edge.Cuts) (width 0.2))
+  (gr_circle (center 260.383754 53.171654) (end 261.383754 53.171654) (layer Edge.Cuts) (width 0.2))
+  (gr_circle (center 194.238754 10.271751) (end 195.238754 10.271751) (layer Edge.Cuts) (width 0.2))
+  (gr_circle (center 74.04084 10.271751) (end 75.04084 10.271751) (layer Edge.Cuts) (width 0.2))
+  (gr_circle (center 74.04084 96.071557) (end 75.04084 96.071557) (layer Edge.Cuts) (width 0.2))
+  (gr_circle (center 194.238754 96.071557) (end 195.238754 96.071557) (layer Edge.Cuts) (width 0.2))
 )
